File: Hardware/Panel/ao_output_panel/ao_output_panel.kicad_pcb (KiCad board)
At the start: 2 copper layers, 100 x 200 mm, 22 parts

Commit message: rm Barton Daughterboard directory; final changes before fabbing; Gerbers; docs updates
Parts:
- removed G***: LOGO, stereo_outs_panel:stereo_outs_panel_art
- removed G***: LOGO, stereo_outs_panel:stereo_outs_panel_holes
- removed the H10 at (132.0, 73.0)
- removed the H11 at (97.0, 103.0)
- removed the H12 at (97.0, 73.0)
- removed the H9 at (132.0, 103.0)
- added GRAF1: Holes, ao_output_panel:ao_output_panel_slide_holes, F.Cu at (100.0, 120.0)
- added GRAF2: Art, ao_output_panel:ao_output_panel_slide_art, F.Cu at (100.0, 120.0)
- added H17: MountingHole_Pad, Kosmo_panel:Kosmo_Panel_Mounting_Hole, F.Cu at (62.5, 37.0)
- added H18: MountingHole_Pad, Kosmo_panel:Kosmo_Panel_Mounting_Hole, F.Cu at (62.5, 117.0)
- added H19: MountingHole_Pad, Kosmo_panel:Kosmo_Panel_Mounting_Hole, F.Cu at (137.5, 37.0)
- added H20: MountingHole_Pad, Kosmo_panel:Kosmo_Panel_Mounting_Hole, F.Cu at (137.5, 117.0)
- moved H1 127.0 mm to (62.5, 170.0)
- moved H9 104.0 mm to (87.5, 137.0)
- moved H2 99.6 mm to (87.5, 170.0)
- moved H3 98.7 mm to (137.5, 170.0)
- moved H10 95.3 mm to (112.5, 137.0)
- moved H4 62.1 mm to (62.5, 195.0)
- moved H8 34.7 mm to (62.5, 137.0)
- moved H5 22.5 mm to (87.5, 195.0)
- moved H12 20.7 mm to (112.5, 170.0)
- moved H6 15.5 mm to (112.5, 195.0)
- moved H11 6.80 mm to (137.5, 137.0)
- moved H7 5.50 mm to (137.5, 195.0)
- renumbered H14 to H10, H15 to H11, H16 to H12, H17 to H13, H18 to H14, H19 to H15, H20 to H16, H13 to H9
Other:
- outline, holes or cut-outs redrawn
- rule pad_to_mask_clearance: 0.05 -> 0
- board text added: "Panel design Rich Holmes Mar 2021"
- board text removed: "Panel design Rich Holmes Sep 2020"
